File: interface-module/interface-module.kicad_sch (KiCad schematic)
At the start: 10 parts, among them J1 Conn_01x08, J2 Conn_01x08, J3 Conn_01x02, SW1 SW_Coded_SH-7050

Commit message: imported I2C, ADC and outputs
Parts:
- removed J1: Conn_01x08, footprints:TerminalBlock_CUI-8_P5.08mm, symbol Connector_Generic:Conn_01x08
- U1: value ~ -> (none)
