File: g0b1re/mints-g0b1re/mints-g0b1re.kicad_sch (KiCad schematic)
At the start: 1 part, among them U1 STM32G0B1RETx

Commit message: Regulator, tranciever, and mcu
Added the regulator, tranciever and mcu to the schematic.
Parts:
- added C1: 10u, symbol Device:C
- added C2, C3: 22u, symbol Device:C
- added C4, C5, C6, C7: 0.1u, symbol Device:C
- added C8: 1n, symbol Device:C
- added D1: LED, symbol Device:LED
- added L1: L, symbol Device:L
- added R1, R2: 10k, symbol Device:R
- added R3, R4: 60.4, symbol Device:R
- added U2: AP63203WU, Package_TO_SOT_SMD:TSOT-23-6, symbol Regulator_Switching:AP63203WU
- added U3: TCAN332, symbol Interface_CAN_LIN:TCAN332
Connections:
- net +3V3: now reaches U1.8 (VDD)
- net +3V3: now also C2.1, C3.1, C5.1, C6.1, C7.1, L1.2, R2.2, U2.1 (FB), U3.3 (VCC)
- new net: C1.2, C2.2, C3.2, U2.4 (GND)
- new net: C8.1, R3.2, R4.2
- new net: C4.2, L1.1, U2.5 (SW)
- new net: C4.1, U2.6 (BST)
- new net: D1.2 (A), R2.1
- new net CAN +: R3.1, U3.7 (CANH)
- new net CAN -: R4.1, U3.6 (CANL)
- new net GND: C5.2, C6.2, C7.2, C8.2, D1.1 (K), U3.2 (GND)
- new net PC4: U3.4 (RXD)
- new net PC5: U3.1 (TXD)
- new net PWR_EN: R1.2, U2.2 (EN)
- new net VBUS: C1.1, R1.1, U2.3 (IN)
- no-connect marks 0 -> 1
Other:
- note added: "3v3 Regulator"
- note added: "CAN Tranceiver"
- note added: "Microcontroller"
- note added: "Random cap 3v3 to gnd in older sheet?"
- note added: "VDDA missing?"
- note added: "what is the purpose of the 10k resistor?"
- company: (none) -> Portland State Aerospace Society
- title: (none) -> Mints Scada Hardware

Commit message: Add CAN bus addr switch, decoupling cap for CAN
Parts:
- added C9: 0.1u, symbol Device:C
- added SW1: SW_Coded_SH-7050, symbol Switch:SW_Coded_SH-7050
Connections:
- net +3V3: now also C9.1, SW1.C
- net GND: now also U1.9 (VSS), C9.2
- net PC4: now also U1.25 (PC4)
- net PC5: now also U1.26 (PC5)
- net at U1.21 (PA4): now also SW1.4
- net at U1.22 (PA5): now also SW1.1
- net at U1.23 (PA6): now also SW1.8
- net at U1.24 (PA7): now also SW1.2
Other:
- note added: "ADDR_1"
- note added: "ADDR_2"
- note added: "ADDR_4"
- note added: "ADDR_8"
- note added: "Address Selector"
- note removed: "Random cap 3v3 to gnd in older sheet?"
- note removed: "VDDA missing?"
- note removed: "what is the purpose of the 10k resistor?"

Commit message: Imported I2C, ADC and Outputs
I coppied in anything that I could from the existing schematic. All the
footprints were assigned. Ready for board layout.
Parts:
- removed C1: 10u, symbol Device:C
- removed C2, C3: 22u, symbol Device:C
- removed C4: 0.1u, symbol Device:C
- removed D1: LED, symbol Device:LED
- removed L1: L, symbol Device:L
- removed R1, R2: 10k, symbol Device:R
- removed U2: AP63203WU, Package_TO_SOT_SMD:TSOT-23-6, symbol Regulator_Switching:AP63203WU
- added C11: 10u, Capacitor_SMD:C_0603_1608Metric, symbol Device:C
- added C12, C14: 22u, Capacitor_SMD:C_0603_1608Metric, symbol Device:C
- added C13: 0.1u, Capacitor_SMD:C_0603_1608Metric, symbol Device:C
- added D3: GREEN, LED_SMD:LED_0603_1608Metric, symbol Device:LED
- added F1: 350mA Poly, Fuse:Fuse_1206_3216Metric, symbol Device:Fuse
- added J1, J2: Conn_01x08, footprints:TerminalBlock_CUI-8_P5.08mm, symbol Connector_Generic:Conn_01x08
- added J3: Conn_01x02, TerminalBlock_Phoenix:TerminalBlock_Phoenix_MKDS-1,5-2-5.08_1x02_P5.08mm_Horizontal, symbol Connector_Generic:Conn_01x02
- added L2: 4.7u, Inductor_SMD:L_1210_3225Metric, symbol Device:L
- added R18: 10k, Resistor_SMD:R_0603_1608Metric, symbol Device:R
- added R19: 5k1, Resistor_SMD:R_0603_1608Metric, symbol Device:R
- added U5: AP63203WU, Package_TO_SOT_SMD:TSOT-23-6, symbol Regulator_Switching:AP63203WU
- C5, C6, C7, C8, C9: footprint (none) -> Capacitor_SMD:C_0603_1608Metric
- R3, R4: footprint (none) -> Resistor_SMD:R_0603_1608Metric
- SW1: footprint (none) -> Button_Switch_THT:Nidec_Copal_SH-7010C
- U3: footprint (none) -> Package_SO:SOIC-8_3.9x4.9mm_P1.27mm
Connections:
- net +3V3: now also C12.1, C14.1, L2.2, R19.1, U5.1 (FB)
- net GND: now also U1.7 (VREF+), C11.2, C12.2, C14.2, D3.1 (K), J2.7 (Pin_7), J2.8 (Pin_8), U5.4 (GND)
- net PWR_EN: now also R18.2, U5.2 (EN)
- net VBUS: now also C11.1, F1.1, R18.1, U5.3 (IN)
- net SPI_SCK: now reaches U1.17 (PA0)
- net CTRL: now reaches U1.18 (PA1)
- net SPI_MOSI: now reaches U1.19 (PA2)
- net SPI_MISO: now reaches U1.20 (PA3)
- net CTL_OUT_0: now reaches U1.27 (PB0)
- net CTL_OUT_1: now reaches U1.28 (PB1)
- net CTL_OUT_2: now reaches U1.29 (PB2)
- net I2C_SCL: now reaches U1.37 (PA9/UCPD1_DBCC1)
- net I2C_SDA: now reaches U1.42 (PA10/UCPD1_DBCC2)
- net CTL_OUT_3: now reaches U1.57 (PB3)
- net CTL_OUT_4: now reaches U1.58 (PB4)
- net CTL_OUT_5: now reaches U1.59 (PB5)
- net CTL_OUT_6: now reaches U1.60 (PB6)
- net CTL_OUT_7: now reaches U1.61 (PB7)
- new net: C13.2, L2.1, U5.5 (SW)
- new net: C13.1, U5.6 (BST)
- new net: F1.2, J2.5 (Pin_5), J2.6 (Pin_6)
- new net: D3.2 (A), R19.2
- new net AUX_POW+: J3.1 (Pin_1)
- new net AU_POW -: J3.2 (Pin_2)
- new net CAN+: J2.3 (Pin_3), J2.4 (Pin_4)
- new net CAN-: J2.1 (Pin_1), J2.2 (Pin_2)
- new net OUT0/IN0+: J1.1 (Pin_1)
- new net OUT1/IN0-: J1.2 (Pin_2)
- new net OUT2/IN1+: J1.3 (Pin_3)
- new net OUT3/IN1-: J1.4 (Pin_4)
- new net OUT4/IN2+: J1.5 (Pin_5)
- new net OUT5/IN2-: J1.6 (Pin_6)
- new net OUT6/IN3+: J1.7 (Pin_7)
- new net OUT7/IN3-: J1.8 (Pin_8)
- no-connect marks 1 -> 41
Other:
- added sheet I2C (I2C.kicad_sch)
- added sheet adc (adc.kicad_sch)
- added sheet outputs (outputs.kicad_sch)
- note added: "35v"
- note added: "Config Option 1: ADC"
- note added: "Config Option 2: Outputs"
- note added: "Config Option 3: I2C"
- note added: "Configuration Instructions For 0-3.3V: R_ADC_TOP: 0 R_ADC_BTM: NP R_ADC_POS: 1k R_ADC_NEG: 1k For 0-33V: R_ADC_TOP: 100k R_ADC_BOT: 11k R_ADC_POS: 0 R_ADC_NEG: 1k For 4-20mA: R_ADC_TOP: 0 R_ADC_BOT: 10 R_ADC_POS: 1k R_ADC_NEG: 1k For higher amps: R_ADC_TOP: 0 R_ADC_BOT: NP R_ADC_POS: 1k R_ADC_NEG: 1k R_SHUNT : shunt"
- note added: "External Plug"
- note added: "I2C is NOT isolated"
- note added: "Inputs are NOT isolated"
- note added: "Output Current Limit Each: Max 2.8A continous @ 15C board above ambient Max 6A peak inrush Combined Max 13A continous @ 15C board above ambient"
- note added: "Outputs are electrically isolated"
- note added: "Pick exactly one during assembally Use the same option for all channels Do not assemble other options"
- moved on the sheet: C5, C6, C7, C8, C9, R3, R4, SW1, U1, U3

Commit message: notes from DR
Other:
- note added: "Add header for STLINK V3 Mini"
- note added: "Andrew says to remove blocks and just use whitespace to seperate"
- note added: "Choose good voltae for caps and power/tolerance for resistors and note on schematic (typ "unless otherwise noted")"
- note added: "Inculde max input/output specs in label"
- note added: "Make this 2 identical 4pin connectors rather than one big so can't plug in wrong spot (each has vbus, gnd, can+, can-)"
- note added: "Remove net labels if you're not going to use them"
- note added: "Rename cas CANRX and CANTX"
- note added: "Route USB D+,D-,Gnd to test point"
- note added: "Select correct pin names on STM footprint (right click on pin -> choose pin function)"
- note added: "TODO add expected power supply specs"
- note added: "TODO check that these are the correct pins"
- note added: "TODO design change verify support for 4-28v system power input"
- note added: "TODO name block"
- note added: "Use detachable plug for all connectors See image below"
- note added: "add SWDCLK, SWDIO, GND, 3.3v to test header"
- note added: "add TP and del label"
- note added: "bit order does not matter on PCB"
- note added: "probs not right probably cap to gnd"
- note added: "switch to TCAN3413DDFR"
- note added: "tie vbat to vdd?"

Commit message: post board review schmatic updates
Parts:
- added C15: 0.1u, Capacitor_SMD:C_0603_1608Metric, symbol Device:C
Connections:
- net +3V3: now also U1.6 (VBAT)
- net GND: now also C15.2; no longer U1.7 (VREF+)
- new net: C15.1, U1.7 (VREF+)
- no-connect marks 41 -> 40
Other:
- note added: "PA1 functions: (SPI1_SCK/I2S1_CK, USART2_RTS_DE_CK, TIM2_CH2, USART4_RX, TIM15_CH1N, I2C1_SMBA, EVENTOUT) there is no CTRL"

Commit message: Schematic progress
Swapped s2c chip, changed 8 pin connecters out with 4 pin, added test
point, removed net labels
Parts:
- removed J2: Conn_01x08, footprints:TerminalBlock_CUI-8_P5.08mm, symbol Connector_Generic:Conn_01x08
- removed U3: TCAN332, Package_SO:SOIC-8_3.9x4.9mm_P1.27mm, symbol Interface_CAN_LIN:TCAN332
- added J2, J4, J5: Conn_01x04, symbol Connector_Generic:Conn_01x04
- added TP1: TestPoint, symbol Connector:TestPoint
- added U2: TCAN3414DDFR, TCAN3414DDFR:SOT65P280X110-8N, symbol TCAN3414DDFR:TCAN3414DDFR
Connections:
- net +3V3: now also U2.3 (VCC)
- net CAN +: now also U2.6 (CANL)
- net CAN -: now also U2.7 (CANH)
- net CAN+: now also J5.1 (Pin_1), J5.2 (Pin_2)
- net CAN-: now also J5.3 (Pin_3), J5.4 (Pin_4)
- net GND: now also J4.1 (Pin_1), J4.2 (Pin_2), U2.2 (GND)
- net at F1.2: now also J4.3 (Pin_3), J4.4 (Pin_4)
- net PC4 renamed CANRX
- net CANRX: now also U2.4 (RXD)
- net PC5 renamed CANTX
- net CANTX: now also U2.1 (TXD)
- net PWR_EN: no longer names the net of R18.2, U5.2 (EN)
- net PWR_EN: now also TP1.1
Other:
- note added: "50v"
- note added: "CAN Plug"
- note added: "Input voltage: 3.8-35V"
- note added: "One TP to usb+, one to usb-, and one to gnd"
- note added: "Upgrade to 50v"
- note removed: "35v"
- note removed: "PA1 functions: (SPI1_SCK/I2S1_CK, USART2_RTS_DE_CK, TIM2_CH2, USART4_RX, TIM15_CH1N, I2C1_SMBA, EVENTOUT) there is no CTRL"
- moved on the sheet: C11, C12, C13, C14, C8, C9, D3, F1, J1, J3, L2, R18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
