File: g0b1re/mints-g0b1re/adc.kicad_sch (KiCad schematic)
At the start: 43 parts, among them U101 MCP3464

Commit message: notes from DR
Other:
- note added: "Add LM4040CIM3-2.0 vref IC"
- note added: "Change ADC IC to MCP3565 (talk to Ben)"

Commit message: Finished Schematic
Added STLINK header. Added flash header. Changed ADC. Fixed ESD caps.
Parts:
- added U3: MCP3565RT-E/SFX, UQFN12_SFX_MCH, symbol 2026-08-04_20-03-06:MCP3565RT-E_SFX
Changed lines of the file:
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@@
+	)
+	(symbol
+		(lib_id "2026-08-04_20-03-06:MCP3565RT-E_SFX")
+		(at 245.11 231.14 0)
+		(unit 1)
+		(body_style 1)
+		(exclude_from_sim no)
+		(in_bom yes)
+		(on_board yes)
+		(in_pos_files yes)
+		(dnp no)
+		(fields_autoplaced yes)
+		(property "Reference" "U3"
+			(at 280.416 230.124 0)
+			(show_name no)
+			(do_not_autoplace no)
+			(effects
+				(font
+					(size 1.524 1.524)
+				)
+			)
+		)
+		(property "Value" "MCP3565RT-E/SFX"
+			(at 280.416 232.664 0)
+			(show_name no)
+			(do_not_autoplace no)
+			(effects
+				(font
+					(size 1.524 1.524)
+				)
+			)
+		)
+		(property "Footprint" "UQFN12_SFX_MCH"
+			(at 237.49 236.22 0)
+			(hide yes)
+			(show_name no)
+			(do_not_autoplace no)
+			(effects
+				(font
+					(size 1.27 1.27)
+					(italic yes)
+				)
+			)
+		)
+		(property "Datasheet" "MCP3565RT-E/SFX"
+			(at 237.49 236.22 0)
+			(hide yes)
+			(show_name no)
+			(do_not_autoplace no)
+			(effects
+				(font
+					(size 1.27 1.27)
+					(italic yes)
+				)
+			)
+		)
+		(property "Description" ""
+			(at 245.11 231.14 0)
+			(hide yes)
+			(show_name no)
+			(do_not_autoplace no)
+			(effects
+				(font
+					(size 1.27 1.27)
+				)
+			)
+		)
+		(pin "7"
+		)
+		(pin "12"
+		)
+		(pin "8"
+		)
+		(pin "11"
+		)
+		(pin "5"
+		)
+		(pin "9"
+		)
+		(pin "13"
+		)
+		(pin "6"
+		)
+		(pin "2"
+		)
+		(pin "4"
+		)
+		(pin "1"
+		)
+		(pin "3"
+		)
+		(pin "10"
+		)
+		(instances
+			(project "mints-g0b1re"
+				(path "/363c6546-315b-48da-9312-6a55f2557799/28c8dc0b-dbda-493a-a6b9-483d7baa93ce"
+					(reference "U3")
+					(unit 1)
+				)
+			)
+		)
 	)
 	(symbol

Commit message: Finished Schematic (missed save)
Same updates from previous commit.
Parts:
- removed C105: 10u, Capacitor_SMD:C_0603_1608Metric, symbol Device:C
- removed C106: 0.1u, Capacitor_SMD:C_0603_1608Metric, symbol Device:C
- removed R103: 0, Resistor_SMD:R_0603_1608Metric, symbol Device:R
- removed U101: MCP3464, Package_DFN_QFN:UQFN-20-1EP_3x3mm_P0.4mm_EP1.85x1.85mm, symbol MCP3464:MCP3464
- removed U3: MCP3565RT-E/SFX, UQFN12_SFX_MCH, symbol 2026-08-04_20-03-06:MCP3565RT-E_SFX
- added C20: 22u, symbol Device:C
- added R30: 510, symbol Device:R
- added R31: 0, Resistor_SMD:R_0603_1608Metric, symbol Device:R
- added TP2: TestPoint, symbol Connector:TestPoint
- added U3: MCP3564R, Package_DFN_QFN:UQFN-20-1EP_3x3mm_P0.4mm_EP1.85x1.85mm, symbol MCP3564:MCP3564
- added U6: LM4040CIM3-2.0/NOPB, DBZ3, symbol 2026-08-04_22-47-04:LM4040CIM3-2.0_NOPB
Connections:
- net +3.3VA: now also U3.18 (Dvdd)
- net +3V3: now also R30.1, U3.19 (AVdd)
- net CTRL: now also U3.11 (~{CS})
- net GND: now also R31.1, U3.17 (Dgnd)
- net IN0+: now also U3.3 (IN0+)
- net IN0-: now also U3.4 (IN0-)
- net IN1+: now also U3.5 (IN1+)
- net IN1-: now also U3.6 (IN1-)
- net IN2+: now also U3.7 (IN2+)
- net IN2-: now also U3.8 (IN2-)
- net IN3+: now also U3.9 (IN3+)
- net IN3-: now also U3.10 (IN3-)
- net SPI_MISO: now also U3.14 (SDO)
- net SPI_MOSI: now also U3.13 (SDI)
- net SPI_SCK: now also U3.12 (SCK)
- net at TP201.1: now also U3.16 (MCLK)
- new net: C20.2, R31.2, TP2.1, U3.1 (REFIN-), U3.20 (Agnd), U3.21 (PAD), U6.2
- new net: C20.1, R30.2, U3.2 (REFIN+), U6.1
- new net EXTI: U3.15 (~{IRQ}/MDAT)
- no-connect marks 1 -> 0
Other:
- note added: "10v"
- moved on the sheet: TP201
