File: g0b1re/mints-g0b1re/_restore_backup_2026-08-13T12-16-53-708/adc.kicad_sch (KiCad schematic)
At the start: 45 parts, among them U3 MCP3564R, U6 LM4040CIM3-2.0/NOPB

Commit message: Board updates
Parts:
- TP2: footprint oresat-misc:TestPoint-0.75mm-th -> (none)
- U6: footprint LM4040CIM3:DBZ3 -> (none)
Changed lines of the file:
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@@
 			)
 		)
-		(property "Footprint" "oresat-misc:TestPoint-0.75mm-th"
+		(property "Footprint" ""
 			(at 287.02 196.85 0)
 			(hide yes)
@@
 			)
 		)
-		(property "Footprint" "LM4040CIM3:DBZ3"
+		(property "Footprint" ""
 			(at 336.296 193.548 0)
 			(hide yes)
