File: g0b1re/mints-g0b1re/_restore_backup_2026-08-13T12-16-53-708/mints-g0b1re.kicad_sch (KiCad schematic)
At the start: 34 parts, among them J1 Conn_01x08, J3 Conn_01x02, J4 Conn_01x04, J5 Conn_01x04, J6 FTSH-107-01-X-DV-K, J7 Conn_01x04, SW1 SW_Coded_SH-7050, U1 STM32G0B1RETx, U2 TCAN3414DDFR, U5 AP63203WU

Commit message: Board updates
Parts:
- removed H1, H2, H3, H4: MountingHole, MountingHole:MountingHole_3.2mm_M3, symbol Mechanical:MountingHole
- D2: footprint LED_SMD:LED_0603_1608Metric -> (none)
- J1: footprint Connector_PinHeader_2.54mm:PinHeader_1x08_P2.54mm_Vertical -> footprints:TerminalBlock_CUI-8_P5.08mm
- J4, J5, J7: footprint Connector_PinHeader_2.54mm:PinHeader_1x04_P2.54mm_Vertical -> (none)
- J6: footprint FTSH:SAMTEC_FTSH-107-01-X-DV-K -> FTSH-107-01-X-DV-K:SAMTEC_FTSH-107-01-X-DV-K
- TP1: footprint oresat-misc:TestPoint-0.75mm-th -> (none)
- U2: footprint TCAN3414DDFR(1):SOT65P280X110-8N -> TCAN3414DDFR:SOT65P280X110-8N
Other:
- moved on the sheet: J1, J3
