File: g0b1re/mints-g0b1re/_restore_backup_2026-08-13T12-16-53-708/outputs.kicad_sch (KiCad schematic)
At the start: 50 parts, among them Q1 SQM120P06-07L_GE3, Q2 SQM120P06-07L_GE3, Q3 SQM120P06-07L_GE3, Q4 SQM120P06-07L_GE3, Q5 SQM120P06-07L_GE3, Q6 SQM120P06-07L_GE3, Q7 SQM120P06-07L_GE3, Q8 SQM120P06-07L_GE3, U201 140357145200, U202 140357145200, U203 140357145200, U204 140357145200, U205 140357145200, U206 140357145200, U207 140357145200, U208 140357145200

Commit message: Board updates
Parts:
- D1: footprint LED_SMD:LED_0603_1608Metric -> (none)
- Q1, Q2, Q3, Q4, Q5, Q6, Q7, Q8: footprint SQM120P06-07L_GE3:TO-263_SQM120P06-07L_GE3_VIS -> (none)
Changed lines of the file:
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@@
 			)
 		)
-		(property "Footprint" "SQM120P06-07L_GE3:TO-263_SQM120P06-07L_GE3_VIS"
+		(property "Footprint" ""
 			(at 209.55 161.29 0)
 			(hide yes)
@@
 			)
 		)
-		(property "Footprint" "SQM120P06-07L_GE3:TO-263_SQM120P06-07L_GE3_VIS"
+		(property "Footprint" ""
 			(at 209.55 119.38 0)
 			(hide yes)
@@
 			)
 		)
-		(property "Footprint" "SQM120P06-07L_GE3:TO-263_SQM120P06-07L_GE3_VIS"
+		(property "Footprint" ""
 			(at 209.55 77.47 0)
 			(hide yes)
@@
 			)
 		)
-		(property "Footprint" "SQM120P06-07L_GE3:TO-263_SQM120P06-07L_GE3_VIS"
+		(property "Footprint" ""
 			(at 167.64 55.88 0)
 			(hide yes)
@@
 			)
 		)
-		(property "Footprint" "SQM120P06-07L_GE3:TO-263_SQM120P06-07L_GE3_VIS"
+		(property "Footprint" ""
 			(at 166.37 182.88 0)
 			(hide yes)
@@
 			)
 		)
-		(property "Footprint" "SQM120P06-07L_GE3:TO-263_SQM120P06-07L_GE3_VIS"
+		(property "Footprint" ""
 			(at 166.37 99.06 0)
 			(hide yes)
@@
 			)
 		)
-		(property "Footprint" "SQM120P06-07L_GE3:TO-263_SQM120P06-07L_GE3_VIS"
+		(property "Footprint" ""
 			(at 166.37 140.97 0)
 			(hide yes)
@@
 			)
 		)
-		(property "Footprint" "LED_SMD:LED_0603_1608Metric"
+		(property "Footprint" ""
 			(at 312.42 95.25 0)
 			(hide yes)
@@
 			)
 		)
-		(property "Footprint" "SQM120P06-07L_GE3:TO-263_SQM120P06-07L_GE3_VIS"
+		(property "Footprint" ""
 			(at 209.55 203.2 0)
 			(hide yes)
